File: kicad/PoolController v1.0.kicad_pcb (KiCad board)
At the start: 2 copper layers, 120 x 100 mm, 61 parts, among them J1 Pompe Péristaltique, J2 Pompe Péristaltique, J4 Sonde température DS18B20, J5 Contacteur Puissance Filtrati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, J6 Conn_01x03, J7 Conn_01x03, J8 Contacteur Puissance Eclairage, J9 Alimentation 12V (2A min), Q2 IRLZ44N, Q4 IRLZ44N, Q5 IRF4905, Q6 IRLZ44N, Q7 IRLZ44N, U1 LM7805_TO220, U2 ESP32-DevKitC, U3 D24V10F3

Commit message: feat: amélioration wizard et minification professionnelle
- Remplacement de minify.py par minify.js avec outils professionnels
  - html-minifier-terser pour HTML
  - Terser pour JavaScript
  - CleanCSS pour CSS
  - Économie: ~92KB / 15% sur le filesystem

- Nouvelle interface de configuration WiFi (wifi.html)
  - Scan des réseaux avec sélection visuelle
  - Validation longueur SSID/password
  - Désactivation automatique du mode AP après connexion
  - Redirection automatique vers http://poolcontroller.local

- Amélioration wizard de configuration initiale
  - Initialisation automatique de l'heure avec heure du navigateur
  - Messages plus clairs après configuration WiFi
  - Persistence du flag wizardCompleted en NVS
  - Correction erreur NVS key length (auth_force_cfg)

- Authentification améliorée
  - Support session token via X-Auth-Token header
  - Exception pour /save-config pendant firstBoot
  - Bouton event listener pour configuration WiFi depuis paramètres

- Documentation mise à jour
  - README.md: outils de build documentés
  - package.json: métadonnées et scripts npm
  - Page "À propos": section outils de build ajoutée

🤖 Generated with [Claude Code](https://claude.com/claude-code)

Co-Authored-By: Claude Sonnet 4.5 <noreply@anthropic.com>
Parts:
- moved C1 240.0 mm to (138.5, 195.7)
- moved J6 240.0 mm to (126.4, 177.0)
- moved R1 240.0 mm to (90.9, 161.7)
Changed lines of the file:
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@@
 	(footprint "Resistor_THT:R_Axial_DIN0207_L6.3mm_D2.5mm_P10.16mm_Horizontal"
 		(layer "F.Cu")
-		(at -118.92 45.21)
+		(at 90.9 161.685)
 		(descr "Resistor, Axial_DIN0207 series, Axial, Horizontal, pin pitch=10.16mm, 0.25W = 1/4W, length*diameter=6.3*2.5mm^2, http://cdn-reichelt.de/documents/datenblatt/B400/1_4W%23YAG.pdf")
 		(tags "Resistor Axial_DIN0207 series Axial Horizontal pin pitch 10.16mm 0.25W = 1/4W length 6.3mm diameter 2.5mm")
@@
 	(footprint "TerminalBlock_Altech:Altech_AK100_1x03_P5.00mm"
 		(layer "F.Cu")
-		(at -83.46 60.525)
+		(at 126.36 177)
 		(descr "Terminal block Altech AK100, 3 pins, pitch 5mm, size 15x9mm, drill diameter 1.3mm, pad diameter 3mm, https://www.altechcorp.com/PDFS/PCBMETRC.PDF#page=3, generated with kicad-footprint-generator TerminalBlock_Altech")
 		(tags "THT Terminal block Altech AK100 pitch 5mm size 15x9mm drill 1.3mm pad 3mm")
@@
 	(footprint "Capacitor_THT:C_Disc_D3.8mm_W2.6mm_P2.50mm"
 		(layer "F.Cu")
-		(at -71.3 79.2)
+		(at 138.52 195.675)
 		(descr "C, Disc series, Radial, pin pitch=2.50mm, diameter*width=3.8*2.6mm^2, Capacitor, http://www.vishay.com/docs/45233/krseries.pdf")
 		(tags "C Disc series Radial pin pitch 2.50mm diameter 3.8mm width 2.6mm Capacitor")

Commit message: feat: ajoute support RTC DS1307 et améliore UI heure
- Ajout du gestionnaire RTC (rtc_manager.cpp/h) avec mutex I2C
- Synchronisation automatique RTC depuis NTP
- Mise à jour RTC lors du réglage manuel de l'heure
- UI: spinner pendant synchronisation NTP
- UI: masquage des secondes sauf en édition manuelle
- UI: rafraîchissement de l'heure synchronisé avec les minutes
- KiCad: mise à jour PCB v1.0 avec fichiers Gerber

Co-Authored-By: Claude Opus 4.5 <noreply@anthropic.com>
Parts:
- removed U1: LM7805_TO220, Package_TO_SOT_THT:TO-220-3_Vertical
- added C21: 10 µF, Capacitor_THT:C_Disc_D6.0mm_W4.4mm_P5.00mm, F.Cu at (62.7, 55.1)
- added C22: 100nF, Capacitor_THT:C_Disc_D3.8mm_W2.6mm_P2.50mm, F.Cu at (62.7, 60.8)
- added C23: 10 µF, Capacitor_THT:C_Disc_D6.0mm_W4.4mm_P5.00mm, F.Cu at (118.6, 52.5)
- added C24: 100nF, Capacitor_THT:C_Disc_D3.8mm_W2.6mm_P2.50mm, F.Cu at (118.6, 57.6)
- added D1: 1N5245B, Diode_THT:D_DO-35_SOD27_P7.62mm_Horizontal, F.Cu at (118.6, 135.1)
- added FB1: BBPY00321611601Y00, Resistor_SMD:R_1206_3216Metric, F.Cu at (62.7, 65.2)
- added FB2: BBPY00321611601Y00, Resistor_SMD:R_1206_3216Metric, F.Cu at (118.6, 65.2)
- added J11: Conn_01x06_Socket, Connector_PinSocket_2.54mm:PinSocket_1x06_P2.54mm_Vertical, F.Cu at (69.7, 71.0)
- added J3: ADS1115, Connector_PinSocket_2.54mm:PinSocket_1x10_P2.54mm_Vertical, F.Cu at (77.4, 60.9)
- added NT1: NetTie_2, NetTie:NetTie-2_THT_Pad1.0mm, F.Cu at (55.1, 64.0)
- added R19: 4.7KΩ, Resistor_THT:R_Axial_DIN0207_L6.3mm_D2.5mm_P10.16mm_Horizontal, F.Cu at (64.0, 79.2)
- added R20: 4.7KΩ, Resistor_THT:R_Axial_DIN0207_L6.3mm_D2.5mm_P10.16mm_Horizontal, F.Cu at (64.0, 75.4)
- added R6: 10KΩ, Resistor_THT:R_Axial_DIN0207_L6.3mm_D2.5mm_P10.16mm_Horizontal, F.Cu at (65.2, 71.6)
- added SW1: B3F-1000, Button_Switch_THT:SW_PUSH_6mm, F.Cu at (79.2, 118.0)
- added U4: OKI-78SR-5_1.5-W36-C, Converter_DCDC:Converter_DCDC_Murata_OKI-78SR_Vertical, F.Cu at (93.2, 131.3)
- C3: value 10 µF -> 100nF
- R1: value 100Ω -> 1KΩ
- moved J1 269.2 mm to (164.5, 73.5), turned to 90 degrees
- moved J2 269.2 mm to (164.5, 84.6), turned to 90 degrees
- moved J5 269.2 mm to (164.5, 95.6), turned to 90 degrees
- moved J8 269.1 mm to (164.5, 106.7), turned to 90 degrees
- moved R15 258.6 mm to (138.9, 105.9), turned to 180 degrees
- moved R13 258.1 mm to (138.9, 90.6), turned to 180 degrees
- moved R16 258.1 mm to (138.9, 100.8), turned to 180 degrees
- moved R7 258.0 mm to (138.9, 75.4), turned to 180 degrees
- moved R5 257.9 mm to (138.9, 55.1), turned to 180 degrees
- moved R14 257.8 mm to (138.9, 85.6), turned to 180 degrees
- moved R4 257.8 mm to (138.9, 60.2), turned to 180 degrees
- moved R8 257.8 mm to (138.9, 70.3), turned to 180 degrees
- moved D7 237.4 mm to (151.5, 116.0), turned to 90 degrees
- moved D6 236.9 mm to (151.6, 100.8), turned to 90 degrees
- moved D2 236.8 mm to (151.6, 70.3), turned to 90 degrees
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Connections:
- C1 pad 2: GND -> GND_ANA
- C10 pad 1: +5V -> Net-(U4-OUT)
- C10 pad 2: GND -> GND_PWR
- C11 pad 2: GND -> GND_PWR
- C12 pad 1: GND -> GND_ANA
- C13 pad 1: +3.3V -> +3.3V_PWR
- C13 pad 2: GND -> GND_PWR
- C14 pad 1: +3.3V -> +3.3V_PWR
- C14 pad 2: GND -> GND_PWR
- C15 pad 1: Net-(D5-A2) -> +12V
- C15 pad 2: GND -> GND_PWR
- C16 pad 1: Net-(D5-A2) -> +12V
- C16 pad 2: GND -> GND_PWR
- C17 pad 2: GND -> GND_PWR
- C18 pad 2: GND -> GND_PWR
- C19 pad 2: GND -> GND_PWR
- C2 pad 1: GND -> GND_PWR
- C2 pad 2: +3.3V -> +3.3V_PWR
- C20 pad 2: GND -> GND_PWR
- C4 pad 2: GND -> GND_PWR
- C5 pad 2: GND -> GND_PWR
- C6 pad 2: GND -> GND_PWR
- C7 pad 2: GND -> GND_PWR
- C8 pad 1: +5V -> Net-(U4-OUT)
- C8 pad 2: GND -> GND_PWR
- C9 pad 2: GND -> GND_PWR
- D5 pad 1: GND -> Net-(D1-K)
- D5 pad 2: Net-(D5-A2) -> GND_PWR
- F1 pad 1: +12V -> Net-(J9-Pin_1)
- F1 pad 2: Net-(D5-A2) -> Net-(D1-K)
- J4 pad 1: GND -> GND_ANA
- J6 pad 2: GND -> GND_ANA
- J7 pad 2: GND -> GND_ANA
- J9 pad 1: +12V -> Net-(J9-Pin_1)
- J9 pad 2: GND -> GND_PWR
- Q2 pad 3: GND -> GND_PWR
- Q4 pad 3: GND -> GND_PWR
- Q5 pad 3: Net-(D5-A2) -> Net-(D1-K)
- Q6 pad 3: GND -> GND_PWR
- Q7 pad 3: GND -> GND_PWR
- R11 pad 1: Net-(D5-A2) -> Net-(D1-K)
- R12 pad 2: GND -> GND_PWR
- R14 pad 2: GND -> GND_PWR
- R16 pad 2: GND -> GND_PWR
- R3 pad 2: GND -> GND_ANA
- R5 pad 2: GND -> GND_PWR
- R8 pad 2: GND -> GND_PWR
- U2 pad 1: +3.3V -> +3.3V_PWR
- U2 pad 10: unconnected-(U2-DAC_2/ADC2_CH9/GPIO26-Pad10) -> /ECLAIRAGE_A2
- U2 pad 12: /POMPE_2 -> unconnected-(U2-MTMS/GPIO14/ADC2_CH6-Pad12)
- U2 pad 14: GND -> GND_PWR
- U2 pad 15: /POMPE_1 -> unconnected-(U2-MTCK/GPIO13/ADC2_CH4-Pad15)
- U2 pad 29: unconnected-(U2-GPIO5-Pad29) -> /DATA_DS18B20
- U2 pad 3: unconnected-(U2-SENSOR_VP/GPIO36/ADC1_CH0-Pad3) -> /RTC_INT
- U2 pad 30: /FILTRATION_A2 -> /POMPE_1
- U2 pad 31: /ECLAIRAGE_A2 -> /POMPE_2
- U2 pad 32: GND -> GND_PWR
- U2 pad 33: unconnected-(U2-GPIO21-Pad33) -> /SDA
- U2 pad 36: unconnected-(U2-GPIO22-Pad36) -> /SCL
- U2 pad 38: GND -> GND_PWR
- U2 pad 5: /DATA_DS18B20 -> unconnected-(U2-VDET_1/GPIO34/ADC1_CH6-Pad5)
- U2 pad 7: /DATA_PH -> /RESET_BUTTON
- U2 pad 8: /DATA_ORP -> unconnected-(U2-32K_XN/GPIO33/ADC1_CH5-Pad8)
- U2 pad 9: unconnected-(U2-DAC_1/ADC2_CH8/GPIO25-Pad9) -> /FILTRATION_A2
- U3 pad 4: GND -> GND_PWR
- U3 pad 5: +3.3V -> +3.3V_PWR
Routing:
- net +12V: track 0.00 -> 187.9 mm
- net +3.3V_PWR: track 0.00 -> 101.8 mm
- net +3.3V: track 0.06 -> 94.8 mm
- net Net-(U4-OUT): track 0.00 -> 89.3 mm
- net /POMPE_1: track 0.00 -> 64.7 mm, vias 0 -> 2
- net /DATA_DS18B20: track 0.00 -> 58.9 mm
- net /POMPE_2: track 0.00 -> 55.6 mm, vias 0 -> 2
- net /SDA: track 0.00 -> 53.5 mm
- net /FILTRATION_A2: track 0.00 -> 51.3 mm, vias 0 -> 2
- net /SCL: track 0.00 -> 46.7 mm
- net /RTC_INT: track 0.00 -> 44.2 mm, vias 0 -> 2
- net /ECLAIRAGE_A2: track 0.00 -> 41.7 mm, vias 0 -> 2
- net +5V: track 0.00 -> 28.2 mm
- net /DATA_ORP: track 0.00 -> 24.9 mm
- net Net-(D2-A): track 0.00 -> 23.9 mm
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- added copper zone on F.Cu, net +12V
- added copper zone on B.Cu, net GND_ANA
- added copper zone on B.Cu, net GND_PWR
Other:
- board size 120 x 100 mm -> 119.4 x 119.4 mm
- board text added: "+"
- board text added: "+3.3V"
- board text added: "12V"
- board text added: "DOSAGE 1"
- board text added: "DOSAGE 2"
- board text added: "ECLAIRAGE"
- board text added: "FILTRATION"
- board text added: "MODULE ORP"
- board text added: "MODULE PH"
- board text added: "RTC_INT"
- board text added: "SONDE TEMPERATURE"
