File: kicad/PoolController v1.0.kicad_sch (KiCad schematic)
At the start: 61 parts, among them J1 Pompe Péristaltique, J2 Pompe Péristaltique, J4 Sonde température DS18B20, J5 Contacteur Puissance Filtrati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, J6 Conn_01x03, J7 Conn_01x03, J8 Contacteur Puissance Eclairage, J9 Alimentation 12V (2A min), Q2 IRLZ44N, Q4 IRLZ44N, Q5 IRF4905, Q6 IRLZ44N, Q7 IRLZ44N, U1 LM7805_TO220, U2 ESP32-DevKitC, U3 D24V10F3

Commit message: Chore: Nettoyage fichiers obsolètes et mise à jour .gitignore
- Suppression fichiers obsolètes
  - SIMULATION_GUIDE.md (mode simulation supprimé)
  - quick_update.sh (mise à jour HTTP supprimée)
  - pre_production_check.sh (script obsolète)

- Ajout assets graphiques
  - menu-icon-64.png pour dashboard
  - logo/logo-1024.png (source haute définition)

- Mise à jour .gitignore
  - Suppression règles backup obsolètes
  - Nettoyage entrées inutiles

- Mise à jour schéma KiCad

🤖 Generated with [Claude Code](https://claude.com/claude-code)

Co-Authored-By: Claude Sonnet 4.5 <noreply@anthropic.com>
Parts:
- added J3: ADS1115 Module, symbol Connector_Generic:Conn_01x10
Connections:
- net +3.3V: now also J3.1 (Pin_1)
- net +5V: now also J3.2 (Pin_2)
- net DATA_DS18B20: now also U2.29 (GPIO5); no longer U2.5 (VDET_1/GPIO34/ADC1_CH6)
- net DATA_ORP: now also J3.8 (Pin_8); no longer U2.8 (32K_XN/GPIO33/ADC1_CH5)
- net DATA_PH: now also J3.7 (Pin_7); no longer U2.7 (32K_XP/GPIO32/ADC1_CH4)
- net SDA: now reaches U2.33 (GPIO21)
- net SDA: now also J3.4 (Pin_4)
- net SCL: now reaches U2.36 (GPIO22)
- net SCL: now also J3.3 (Pin_3)
Other:
- note added: "Module ORP Sortie analogique 0 ~ +4V"
- note removed: "Module ORP Sortie analogique 0 ~ +5V"
- moved on the sheet: C1, C10, C11, C12, C13, C14, C15, C16, C17, C18, C19, C20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

Commit message: docs: documentation complète du bouton reset et schéma KiCad
Documentation (QUICK_START.md):
- Ajout section détaillée "Procédure de reset"
- Documentation complète des effets du reset password
- Ajout section "Après le reset" avec workflow complet
- Précisions techniques sur le bouton (NO, pull-up interne)
- Documentation activation automatique mode AP
- Documentation bouton WiFi sur écran login
- Documentation changement obligatoire du mot de passe

Schéma KiCad (PoolController v1.0):
- Ajout convertisseur ADS1115 (ADC 16 bits I2C)
- Ajout bouton Reset (GPIO4 → GND, NO avec pull-up interne)
- Mise à jour du schéma électronique

Le bouton reset réinitialise:
- Mot de passe → admin
- Token API → régénéré
- Active le mode AP WiFi (AP + STA)
- Affiche le bouton "Configurer le Wi-Fi" sur l'écran de login
- Force le changement de mot de passe à la première connexion

🤖 Generated with [Claude Code](https://claude.com/claude-code)

Co-Authored-By: Claude Sonnet 4.5 <noreply@anthropic.com>
Parts:
- added SW1: Bouton Reset, Button_Switch_THT:SW_PUSH_6mm, symbol Switch:SW_Push
- C1: value 100nF -> 10 µF
- J3: value ADS1115 Module -> ADS1115; footprint (none) -> Connector_PinHeader_2.54mm:PinHeader_1x10_P2.54mm_Vertical
- R1: value 100Ω -> 4.7KΩ
Connections:
- net +3.3V: now also SW1.2
- net DATA_ORP: now also U2.5 (VDET_1/GPIO34/ADC1_CH6)
- net DATA_PH: now also U2.6 (VDET_2/GPIO35/ADC1_CH7)
- net RESET_BUTTON: now reaches U2.26 (ADC2_CH0/GPIO4)
- net RESET_BUTTON: now also SW1.1
- no-connect marks 26 -> 21
Other:
- note added: "Convertisseur analogique numérique"
- note added: "R1 & C1 optimisés pour un GAIN_ONE et SDS de 8 sur l'ADS1115"
- note removed: "0 ~ 3.3V"
- moved on the sheet: C1, C10, C11, C12, C13, C14, C15, C16, C17, C18, C19, C20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

Commit message: feat: ajoute support RTC DS1307 et améliore UI heure
- Ajout du gestionnaire RTC (rtc_manager.cpp/h) avec mutex I2C
- Synchronisation automatique RTC depuis NTP
- Mise à jour RTC lors du réglage manuel de l'heure
- UI: spinner pendant synchronisation NTP
- UI: masquage des secondes sauf en édition manuelle
- UI: rafraîchissement de l'heure synchronisé avec les minutes
- KiCad: mise à jour PCB v1.0 avec fichiers Gerber

Co-Authored-By: Claude Opus 4.5 <noreply@anthropic.com>
Parts:
- removed U1: LM7805_TO220, Package_TO_SOT_THT:TO-220-3_Vertical, symbol Regulator_Linear:LM7805_TO220
- added C21, C23: 10 µF, Capacitor_THT:C_Disc_D6.0mm_W4.4mm_P5.00mm, symbol Device:C
- added C22, C24: 100nF, Capacitor_THT:C_Disc_D3.8mm_W2.6mm_P2.50mm, symbol Device:C
- added D1: 1N5245B, Diode_THT:D_DO-35_SOD27_P7.62mm_Horizontal, symbol Device:D_Zener
- added FB1, FB2: BBPY00321611601Y00, Resistor_SMD:R_1206_3216Metric, symbol Device:FerriteBead
- added J11: Conn_01x06_Socket, Connector_PinSocket_2.54mm:PinSocket_1x06_P2.54mm_Vertical, symbol Connector:Conn_01x06_Socket
- added NT1: NetTie_2, NetTie:NetTie-2_THT_Pad1.0mm, symbol Device:NetTie_2
- added R19, R20: 4.7KΩ, Resistor_THT:R_Axial_DIN0207_L6.3mm_D2.5mm_P10.16mm_Horizontal, symbol Device:R
- added R6: 10KΩ, Resistor_THT:R_Axial_DIN0207_L6.3mm_D2.5mm_P10.16mm_Horizontal, symbol Device:R
- added U4: OKI-78SR-5_1.5-W36-C, Converter_DCDC:Converter_DCDC_Murata_OKI-78SR_Vertical, symbol Converter_DCDC:OKI-78SR-5_1.5-W36-C
- C1, C3: value 10 µF -> 100nF
- J3: footprint Connector_PinHeader_2.54mm:PinHeader_1x10_P2.54mm_Vertical -> Connector_PinSocket_2.54mm:PinSocket_1x10_P2.54mm_Vertical
- R1: value 4.7KΩ -> 1KΩ
- SW1: value Bouton Reset -> B3F-1000
Connections:
- net +12V: now also C15.1, C16.1, U4.1 (IN); no longer F1.1, J9.1 (Pin_1)
- net +3.3V: now also C21.1, C22.1, FB1.1, J11.5 (Pin_5); no longer C13.1, C14.1, C2.2, SW1.2, U2.1 (3V3), U3.5 (VOUT)
- net +5V: now also C23.1, C24.1, FB2.1; no longer C1.2, C10.1, C10.2, C11.2, C12.1, C13.2, C14.2, C15.2, C16.2, C17.2, C18.2, C19.2, C2.1, C20.2, C3.1, C3.2, C4.2, C5.2, C6.2, C7.2, C8.1, C8.2, C9.2, D5.1 (A1), J3.2 (Pin_2), J4.1 (Pin_1), J6.2 (Pin_2), J7.2 (Pin_2), J7.3 (Pin_3), J9.2 (Pin_2), Q2.3 (S), Q4.3 (S), Q6.3 (S), Q7.3 (S), R12.2, R14.2, R16.2, R2.1, R3.2, R5.2, R8.2, U2.14 (GND), U2.32 (GND), U2.38 (GND), U3.4 (GND)
- net DATA_ORP: no longer U2.5 (VDET_1/GPIO34/ADC1_CH6)
- net DATA_PH: no longer U2.6 (VDET_2/GPIO35/ADC1_CH7)
- net ECLAIRAGE_A2: now also U2.10 (DAC_2/ADC2_CH9/GPIO26); no longer U2.31 (GPIO19)
- net FILTRATION_A2: now also U2.9 (DAC_1/ADC2_CH8/GPIO25); no longer U2.30 (GPIO18)
- net POMPE_1: now also U2.30 (GPIO18); no longer U2.9 (DAC_1/ADC2_CH8/GPIO25)
- net POMPE_2: now also U2.31 (GPIO19); no longer U2.10 (DAC_2/ADC2_CH9/GPIO26)
- net RESET_BUTTON: now also U2.7 (32K_XP/GPIO32/ADC1_CH4); no longer U2.26 (ADC2_CH0/GPIO4)
- net SCL: now also J11.3 (Pin_3), R20.2
- net SDA: now also J11.4 (Pin_4), R19.2
- net at F1.2, Q5.3 (S), R11.1: now also D5.1 (A1), D1.1 (K); no longer C15.1, C16.1, D5.2 (A2)
- net at Q5.1 (G), R11.2, R12.1: now also D1.2 (A)
- net RTC_INT: now reaches U2.3 (SENSOR_VP/GPIO36/ADC1_CH0)
- net RTC_INT: now also J11.1 (Pin_1), R6.1
- new net: C10.1, C8.1, FB2.2, U4.3 (OUT)
- new net: C3.1, J7.3 (Pin_3), R2.1
- new net: F1.1, J9.1 (Pin_1)
- new net +3.3V_PWR: C13.1, C14.1, C2.2, FB1.2, R19.1, R20.1, R6.2, SW1.2, U2.1 (3V3), U3.5 (VOUT)
- new net GND: C3.2
- new net GND_ANA: C1.2, C12.1, C21.2, C22.2, C23.2, C24.2, J11.6 (Pin_6), J3.2 (Pin_2), J4.1 (Pin_1), J6.2 (Pin_2), J7.2 (Pin_2), NT1.1, R3.2
- new net GND_PWR: C10.2, C11.2, C13.2, C14.2, C15.2, C16.2, C17.2, C18.2, C19.2, C2.1, C20.2, C4.2, C5.2, C6.2, C7.2, C8.2, C9.2, D5.2 (A2), J9.2 (Pin_2), NT1.2, Q2.3 (S), Q4.3 (S), Q6.3 (S), Q7.3 (S), R12.2, R14.2, R16.2, R5.2, R8.2, U2.14 (GND), U2.32 (GND), U2.38 (GND), U3.4 (GND), U4.2 (GND)
- no-connect marks 21 -> 30
Other:
- note added: "Alim 3.3V 1A Module ESP32-WROOM-32 : 250 mA max Module pH : 5-10mA"
- note added: "Diode Zener Protection Gate 15V"
- note added: "Masse en étoile"
- note added: "Module RTC DS3231"
- note removed: "Alim 3.3V 1A Module ESP32-WROOM-32 : 250 mA max Module ORP : ? Module pH : 5-10mA 2 Relais SRD-03VDC-SL-C : 2 * 100 mA"
- moved on the sheet: C1, C10, C11, C12, C13, C14, C15, C16, C17, C18, C19, C20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
